Commit message: latest updates

File: dasl_manipulators/HDT_MK2/mk2_arm_description/robots/mk2_arm_description.URDF (robot description, URDF)
Before this commit: robot mk2_arm_description, 11 links, 10 joints
Links:
- removed link gimbal_pitch_link
- removed link gimbal_roll_link
- removed link gimbal_yaw_link
- removed link right_elbow_pitch_link
- removed link right_shoulder_pitch_link
- removed link right_shoulder_roll_link
- removed link right_shoulder_yaw_link
- removed link right_wrist_pitch_link
- removed link right_wrist_roll_link
- removed link right_wrist_yaw_link
- added link gimbal_pitch_Link, mass 0.214939219832887; collision mesh filename=package://mk2_arm_description/meshes/gimbal_pitch_Link.STL; visual mesh filename=package://mk2_arm_description/meshes/gimbal_pitch_Link.STL
- added link gimbal_roll_Link, mass 0.293335683340013; collision mesh filename=package://mk2_arm_description/meshes/gimbal_roll_Link.STL; visual mesh filename=package://mk2_arm_description/meshes/gimbal_roll_Link.STL
- added link gimbal_yaw_Link, mass 0.312439408979876; collision mesh filename=package://mk2_arm_description/meshes/gimbal_yaw_Link.STL; visual mesh filename=package://mk2_arm_description/meshes/gimbal_yaw_Link.STL
- added link right_elbow_pitch_Link, mass 0.0687829528144863; collision mesh filename=package://mk2_arm_description/meshes/right_elbow_pitch_Link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; visual mesh filename=package://mk2_arm_description/meshes/right_elbow_pitch_Link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
- added link right_index_finger_pitch_Link, mass 0.0194186234284368; collision mesh filename=package://mk2_arm_description/meshes/right_index_finger_pit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; visual mesh filename=package://mk2_arm_description/meshes/right_index_finger_pit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
- added link right_middle_finger_pitch_Link, mass 0.0194186227284907; collision mesh filename=package://mk2_arm_description/meshes/right_middle_finger_pi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; visual mesh filename=package://mk2_arm_description/meshes/right_middle_finger_pi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
- added link right_shoulder_pitch_Link, mass 0.163444561598499; collision mesh filename=package://mk2_arm_description/meshes/right_shoulder_pitch_L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; visual mesh filename=package://mk2_arm_description/meshes/right_shoulder_pitch_L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
- added link right_shoulder_roll_Link, mass 0.0635014734267768; collision mesh filename=package://mk2_arm_description/meshes/right_shoulder_roll_Li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; visual mesh filename=package://mk2_arm_description/meshes/right_shoulder_roll_Li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
- added link right_shoulder_yaw_Link, mass 0.234264117637169; collision mesh filename=package://mk2_arm_description/meshes/right_shoulder_yaw_Lin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; visual mesh filename=package://mk2_arm_description/meshes/right_shoulder_yaw_Lin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
- added link right_thumb_pitch_Link, mass 0.019612487052281; collision mesh filename=package://mk2_arm_description/meshes/right_thumb_pitch_Link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; visual mesh filename=package://mk2_arm_description/meshes/right_thumb_pitch_Link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
- added link right_thumb_roll_Link, mass 0.0873521059346375; collision mesh filename=package://mk2_arm_description/meshes/right_thumb_roll_Link.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; visual mesh filename=package://mk2_arm_description/meshes/right_thumb_roll_Link.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
- added link right_wrist_pitch_Link, mass 0.0439051251849098; collision mesh filename=package://mk2_arm_description/meshes/right_wrist_pitch_Link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; visual mesh filename=package://mk2_arm_description/meshes/right_wrist_pitch_Link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
- added link right_wrist_roll_Link, mass 0.366836124330785; collision mesh filename=package://mk2_arm_description/meshes/right_wrist_roll_Link.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; visual mesh filename=package://mk2_arm_description/meshes/right_wrist_roll_Link.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
- added link right_wrist_yaw_Link, mass 0.143237840838415; collision mesh filename=package://mk2_arm_description/meshes/right_wrist_yaw_Link.S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; visual mesh filename=package://mk2_arm_description/meshes/right_wrist_yaw_Link.S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
Joints:
- added joint right_index_finger_pitch_joint: type continuous, parent right_wrist_roll_Link, child right_index_finger_pitch_Link, origin xyz=-0.00196555449049784 -0.218573499999996 0 rpy=1.5707963267949 -0.172649920415237 -1.5707963267949, axis 0 0 1
- added joint right_middle_finger_pitch_joint: type continuous, parent right_wrist_roll_Link, child right_middle_finger_pitch_Link, origin xyz=-0.0233993322569385 0.334555337087318 0.0945748698744839 rpy=1.5707963267949 -0.129408348093935 -1.5707963267949, axis 0 0 1
- added joint right_thumb_pitch_joint: type continuous, parent right_thumb_roll_Link, child right_thumb_pitch_Link, origin xyz=0 -0.0569235000000001 -0.0258516178434754 rpy=3.14159265358979 1.27445866924021 -1.5707963267949, axis 0 -1 0
- added joint right_thumb_roll_joint: type continuous, parent right_wrist_roll_Link, child right_thumb_roll_Link, origin xyz=-0.015284999999999 -0.109781382156522 0 rpy=-1.57079632679516 -1.55914211708858 2.67339782685593E-13, axis 0 0 1
- joint gimbal_pitch_joint: child gimbal_pitch_link -> gimbal_pitch_Link; origin xyz=0 0.1065 0 rpy=-0.0107280632545701 -2.08166817117217E-17 0 -> xyz=0 0.1065 0 rpy=-0.00759652588906983 -2.18575157973078E-16 2.71050543121376E-20; parent gimbal_yaw_link -> gimbal_yaw_Link
- joint gimbal_roll_joint: child gimbal_roll_link -> gimbal_roll_Link; origin xyz=0 0.08 0 rpy=3.29597460435593E-17 5.89805981832114E-17 -0.00720353270271086 -> xyz=0 0.0799999992233969 0 rpy=-3.27862736959617E-16 -6.59194920871187E-17 -0.0104219206899189; parent gimbal_pitch_link -> gimbal_pitch_Link
- joint gimbal_yaw_joint: child gimbal_yaw_link -> gimbal_yaw_Link; origin xyz=0 0 0.0207 rpy=1.5707963267949 -7.62441236410402E-19 -0.0124523433757913 -> xyz=0 0 0.0207 rpy=1.5707963267949 -7.94164081897E-19 -0.0129704757340406
- joint right_elbow_pitch_joint: child right_elbow_pitch_link -> right_elbow_pitch_Link; origin xyz=0 0 -0.245154351351583 rpy=-1.57079632679542 1.56342870700628 -5.24290930743869E-13 -> xyz=0 0 -0.238827805276381 rpy=1.57079632679492 -1.49996318713234 3.14159265358977; parent right_shoulder_yaw_link -> right_shoulder_yaw_Link
- joint right_shoulder_pitch_joint: child right_shoulder_pitch_link -> right_shoulder_pitch_Link; origin xyz=-0.0745159451359152 0.36378233047 0 rpy=-1.57079632679484 -1.5588414942257 -1.57079632679496 -> xyz=-0.0744803728234152 0.363782413385281 0 rpy=1.57079632679489 -1.4781863977047 1.5707963267949; parent gimbal_roll_link -> gimbal_roll_Link
- joint right_shoulder_roll_joint: child right_shoulder_roll_link -> right_shoulder_roll_Link; origin xyz=0 0 -0.175004054864085 rpy=-1.57079632679511 1.5680965801137 1.57079632679469 -> xyz=0 0 -0.175031746128161 rpy=-1.57079632679491 1.53633681961858 1.57079632679488; parent right_shoulder_pitch_link -> right_shoulder_pitch_Link
- joint right_shoulder_yaw_joint: child right_shoulder_yaw_link -> right_shoulder_yaw_Link; origin xyz=0 -0.0728206486484171 0 rpy=1.57079632679491 1.48659895798722 -3.14159265358978 -> xyz=0 -0.0791471947236229 0 rpy=-1.57079632679489 -0.37295399710194 3.20398189477444E-16; parent right_shoulder_roll_link -> right_shoulder_roll_Link
- joint right_wrist_pitch_joint: axis -1 0 0 -> 0 0 1; child right_wrist_pitch_link -> right_wrist_pitch_Link; origin xyz=0 -0.0740999999999999 0 rpy=-1.61133676385665 -1.16985414411186E-16 -8.95117313604032E-16 -> xyz=0 0 -0.176348456415071 rpy=-1.57079632679489 1.51953810704376 1.57079632679491; parent right_wrist_roll_link -> right_wrist_yaw_Link
- joint right_wrist_roll_joint: axis 0 0 -1 -> -1 0 0; child right_wrist_roll_link -> right_wrist_roll_Link; origin xyz=0 0 -0.124475 rpy=1.5707963267949 0.0155767413507828 -0.0165465548293445 -> xyz=0 -0.074100000000003 0 rpy=0.0362653907896615 1.66533453693773E-16 -1.45716771982052E-16; parent right_wrist_yaw_link -> right_wrist_pitch_Link
- joint right_wrist_yaw_joint: axis 0 0 0 -> 0 0 1; child right_wrist_yaw_link -> right_wrist_yaw_Link; origin xyz=0 -0.0999700000000001 0 rpy=3.11921549796857 -1.57079631189374 1.59181711218594 -> xyz=0 -0.048096543584929 0 rpy=1.57079632679489 -1.45958116646768 -3.14159265358979; parent right_elbow_pitch_link -> right_elbow_pitch_Link; type fixed -> continuous
