Commit message: updates to mocap

File: dasl_controllers/mk2_controller/robots/mk2_controller.URDF (robot description, URDF)
Before this commit: robot mk2_gimbal_description, 5 links, 4 joints
Links:
- removed link gantry_link
- removed link gimbal_base_link
- added link gantry_gimbal_base_link, mass 0.356270706990662; collision mesh filename=package://mk2_controller/meshes/gantry_gimbal_base_link.STL; visual mesh filename=package://mk2_controller/meshes/gantry_gimbal_base_link.STL
- link gimbal_pitch_link: mass 0.21494 -> 0.214939217277683
- link gimbal_roll_link: mass 0.29334 -> 0.29333576544646
- link gimbal_yaw_link: mass 0.31244 -> 0.312439397659762
Joints:
- removed joint gantry_joint
- joint gimbal_pitch_joint: origin xyz=0 0.1065 0 rpy=0.015488 0 0 -> xyz=0 0.1065 0 rpy=0.015488 1.1768E-14 -3.0626E-20
- joint gimbal_roll_joint: origin xyz=0 0.08 0 rpy=0 0 0.033714 -> xyz=0 0.08 0 rpy=-2.3375E-16 -1.707E-15 0.033714
- joint gimbal_yaw_joint: origin xyz=0 0 0.0207 rpy=1.5708 0 1.5894 -> xyz=0 0 0.0207 rpy=1.5708 -5.6772E-17 1.5894; parent gimbal_base_link -> gantry_gimbal_base_link

File: dasl_controllers/mk2_controller/robots/mk2_gimbal.URDF (robot description, URDF)
Before this commit: robot mk2_gimbal_description, 5 links, 4 joints
Links:
- removed link gantry_link
- link gimbal_base_link: mass 0.13049 -> 0.130487655760344; geometry collision mesh filename=package://mk2_controller/meshes_v2/gimbal_base_link.STL; visual mesh filename=package://mk2_controller/meshes_v2/gimbal_base_link.STL
- link gimbal_pitch_link: geometry collision mesh filename=package://mk2_controller/meshes_v2/gimbal_pitch_link.STL; visual mesh filename=package://mk2_controller/meshes_v2/gimbal_pitch_link.STL
- link gimbal_roll_link: geometry collision mesh filename=package://mk2_controller/meshes_v2/gimbal_roll_link.STL; visual mesh filename=package://mk2_controller/meshes_v2/gimbal_roll_link.STL
- link gimbal_yaw_link: geometry collision mesh filename=package://mk2_controller/meshes_v2/gimbal_yaw_link.STL; visual mesh filename=package://mk2_controller/meshes_v2/gimbal_yaw_link.STL
Joints:
- removed joint gantry_joint
- joint gimbal_pitch_joint: axis 1 0 0 -> 0 0 0; origin xyz=0 0.1065 0 rpy=0.015488 0 0 -> xyz=0 0 0 rpy=0 2.2956E-49 0
- joint gimbal_roll_joint: axis 0 0 -1 -> 0 0 0; origin xyz=0 0.08 0 rpy=0 0 0.033714 -> xyz=0 0 0 rpy=0 2.2956E-49 0
- joint gimbal_yaw_joint: axis 0 -1 0 -> 0 0 0; origin xyz=0 0 0.0207 rpy=1.5708 0 1.5894 -> xyz=0 0 0 rpy=0 1.5708 0
