Commit message: changes to dae, urdf, simulation

File: dasl_robots/mk2/robots/mk2.URDF (robot description, URDF)
Before this commit: robot mk2, 16 links, 15 joints
Links:
- removed link right_index_finger_link
- removed link right_middle_finger_link
- removed link right_palm_link
- removed link right_thumb_pitch_link
- removed link right_thumb_yaw_link
- removed link torso_base_link
- removed link torso_pitch_link
- removed link torso_yaw_link
- link right_elbow_pitch_link: mass 0.0687829523644407 -> None; geometry visual mesh filename=package://mk2/meshes/right_elbow_pitch_link.STL
- link right_shoulder_pitch_link: mass 0.163443866563097 -> None; geometry visual mesh filename=package://mk2/meshes/right_shoulder_pitch_link.STL
- link right_shoulder_roll_link: mass 0.0635014085130222 -> None; geometry visual mesh filename=package://mk2/meshes/right_shoulder_roll_link.STL
- link right_shoulder_yaw_link: mass 0.234264177667547 -> None; geometry visual mesh filename=package://mk2/meshes/right_shoulder_yaw_link.STL
- link right_wrist_pitch_link: mass 0.0439051251850394 -> None; geometry visual mesh filename=package://mk2/meshes/right_wrist_pitch_link.STL
- link right_wrist_roll_link: mass 0.0825624287077396 -> None; geometry visual mesh filename=package://mk2/meshes/right_wrist_roll_link.STL
- link right_wrist_yaw_link: mass 0.143237901554334 -> None; geometry visual mesh filename=package://mk2/meshes/right_wrist_yaw_link.STL
- link torso_roll_link: mass 0.293335697547887 -> None; geometry visual mesh filename=package://mk2/meshes/torso_roll_link.STL
Joints:
- removed joint right_index_finger_joint
- removed joint right_middle_finger_joint
- removed joint right_palm_joint
- removed joint right_thumb_pitch_joint
- removed joint right_thumb_yaw_joint
- removed joint torso_pitch_joint
- removed joint torso_roll_joint
- removed joint torso_yaw_joint
- joint right_elbow_pitch_joint: axis 0 0 -1 -> 1 0 0; limit (none) -> lower=-1.57 upper=1.57 effort=30 velocity=1.0; origin xyz=0 0 -0.24462 rpy=-1.5708 1.5707 -3.1416 -> xyz=0 -0.24462 0 rpy=0 0 0; type continuous -> revolute
- joint right_shoulder_pitch_joint: axis 0 0 -1 -> 1 0 0; limit (none) -> lower=-1.57 upper=1.57 effort=30 velocity=1.0; origin xyz=-0.0754 0.36378 0 rpy=1.5708 -1.5707 1.5708 -> xyz=-0.0754 0.36378 0 rpy=0 0 0; type continuous -> revolute
- joint right_shoulder_roll_joint: limit (none) -> lower=-0.4 upper=3.14 effort=30 velocity=1.0; origin xyz=0 0 -0.17412 rpy=3.14159265358979 -1.5707963267949 0 -> xyz=-0.17412 0 0 rpy=0 0 0; type continuous -> revolute
- joint right_shoulder_yaw_joint: axis 0 0 1 -> 0 1 0; limit (none) -> lower=-1.57 upper=1.57 effort=30 velocity=1.0; origin xyz=0 -0.0733500255441 0 rpy=-1.57079632679615 1.56889022393905 2.09530269072339E-07 -> xyz=0 -0.073 0 rpy=0 0 0; type continuous -> revolute
- joint right_wrist_pitch_joint: axis 0 0 -1 -> 1 0 0; limit (none) -> lower=-1.57 upper=1.57 effort=30 velocity=1.0; type continuous -> revolute
- joint right_wrist_roll_joint: axis 1 0 0 -> 0 0 1; limit (none) -> lower=-1.57 upper=1.57 effort=30 velocity=1.0; origin xyz=0 -0.0740999999999999 0 rpy=0.00190610286735421 0 0 -> xyz=0 -0.07 0 rpy=0 0 0; type continuous -> revolute
- joint right_wrist_yaw_joint: axis 0 -1 0 -> 0 1 0; limit (none) -> lower=-1.57 upper=1.57 effort=30 velocity=1.0; origin xyz=0 0.0732006015482298 0 rpy=1.30104260698261E-18 -1.16246228532812E-19 3.14159265358979 -> xyz=0 -0.0732 0 rpy=0 0 0; type continuous -> revolute

Commit message: major updates to model

File: dasl_robots/mk2/robots/mk2.URDF (robot description, URDF)
Before this commit: robot mk2, 8 links, 7 joints
Links:
- added link right_index_yaw_link, mass 0.0183440339634614; collision mesh filename=package://mk2/meshes/right_index_yaw_link.STL; visual mesh filename=package://mk2/meshes/right_index_yaw_link.STL
- added link right_palm_link, mass 0.28427392143233; collision mesh filename=package://mk2/meshes/right_palm_link.STL; visual mesh filename=package://mk2/meshes/right_palm_link.STL
- added link right_ring_yaw_link, mass 0.0183440282672802; collision mesh filename=package://mk2/meshes/right_ring_yaw_link.STL; visual mesh filename=package://mk2/meshes/right_ring_yaw_link.STL
- added link right_thumb_pitch_link, mass 0.0183440323230481; collision mesh filename=package://mk2/meshes/right_thumb_pitch_link.STL; visual mesh filename=package://mk2/meshes/right_thumb_pitch_link.STL
- added link right_thumb_roll_link, mass 0.0873520694654447; collision mesh filename=package://mk2/meshes/right_thumb_roll_link.STL; visual mesh filename=package://mk2/meshes/right_thumb_roll_link.STL
- added link torso_base_link, mass 0.130487655760344; collision mesh filename=package://mk2/meshes/torso_base_link.STL; visual mesh filename=package://mk2/meshes/torso_base_link.STL
- added link torso_pitch_link, mass 0.214939253072605; collision mesh filename=package://mk2/meshes/torso_pitch_link.STL; visual mesh filename=package://mk2/meshes/torso_pitch_link.STL
- added link torso_yaw_link, mass 0.312439405406118; collision mesh filename=package://mk2/meshes/torso_yaw_link.STL; visual mesh filename=package://mk2/meshes/torso_yaw_link.STL
- link right_elbow_pitch_link: mass None -> 0.0687829534109835; geometry collision mesh filename=package://mk2/meshes/right_elbow_pitch_link.STL; visual mesh filename=package://mk2/meshes/right_elbow_pitch_link.STL
- link right_shoulder_pitch_link: mass None -> 0.140151957793056; geometry collision mesh filename=package://mk2/meshes/right_shoulder_pitch_link.STL; visual mesh filename=package://mk2/meshes/right_shoulder_pitch_link.STL
- link right_shoulder_roll_link: mass None -> 0.06350140855047; geometry collision mesh filename=package://mk2/meshes/right_shoulder_roll_link.STL; visual mesh filename=package://mk2/meshes/right_shoulder_roll_link.STL
- link right_shoulder_yaw_link: mass None -> 0.234264171591375; geometry collision mesh filename=package://mk2/meshes/right_shoulder_yaw_link.STL; visual mesh filename=package://mk2/meshes/right_shoulder_yaw_link.STL
- link right_wrist_pitch_link: mass None -> 0.0439051251849812; geometry collision mesh filename=package://mk2/meshes/right_wrist_pitch_link.STL; visual mesh filename=package://mk2/meshes/right_wrist_pitch_link.STL
- link right_wrist_roll_link: mass None -> 0.143237868675615; geometry collision mesh filename=package://mk2/meshes/right_wrist_roll_link.STL; visual mesh filename=package://mk2/meshes/right_wrist_roll_link.STL
- link right_wrist_yaw_link: mass None -> 0.0825624287077141; geometry collision mesh filename=package://mk2/meshes/right_wrist_yaw_link.STL; visual mesh filename=package://mk2/meshes/right_wrist_yaw_link.STL
- link torso_roll_link: mass None -> 0.293335697547887; geometry collision mesh filename=package://mk2/meshes/torso_roll_link.STL; visual mesh filename=package://mk2/meshes/torso_roll_link.STL
Joints:
- added joint right_index_yaw_joint: type revolute, parent right_palm_link, child right_index_yaw_link, origin xyz=0.0696 0 0.0193 rpy=0 0 0, axis 0 0 1, limit lower=-1.57 upper=1.57 effort=10 velocity=1.0
- added joint right_palm_joint: type fixed, parent right_wrist_yaw_link, child right_palm_link, origin xyz=0.1489 0 0 rpy=0 0 0, axis 0 0 0
- added joint right_ring_yaw_joint: type revolute, parent right_palm_link, child right_ring_yaw_link, origin xyz=0.0696 0 -0.0039 rpy=0 0 0, axis 0 0 1, limit lower=-1.57 upper=1.57 effort=10 velocity=1.0
- added joint right_thumb_pitch_joint: type revolute, parent right_thumb_roll_link, child right_thumb_pitch_link, origin xyz=-0.013307 0 0.05692 rpy=0 0 0, axis 0 1 0, limit lower=-1.57 upper=1.57 effort=10 velocity=1.0
- added joint right_thumb_roll_joint: type revolute, parent right_palm_link, child right_thumb_roll_link, origin xyz=0 0 0.0153 rpy=0 0 0, axis 1 0 0, limit lower=-1.57 upper=1.57 effort=10 velocity=1.0
- added joint torso_pitch_joint: type revolute, parent torso_yaw_link, child torso_pitch_link, origin xyz=0 0 -0.1065 rpy=0 0 0, axis 0 -1 0, limit lower=-1.57 upper=1.57 effort=10 velocity=1.0
- added joint torso_roll_joint: type revolute, parent torso_pitch_link, child torso_roll_link, origin xyz=0 0 -0.08 rpy=0 0 0, axis 1 0 0, limit lower=-1.57 upper=1.57 effort=10 velocity=1.0
- added joint torso_yaw_joint: type revolute, parent torso_base_link, child torso_yaw_link, origin xyz=0 0 -0.0207 rpy=0 0 0, axis 0 0 -1, limit lower=-1.57 upper=1.57 effort=10 velocity=1.0
- joint right_elbow_pitch_joint: axis 1 0 0 -> 0 1 0; limit lower=-1.57 upper=1.57 effort=30 velocity=1.0 -> lower=-1.57 upper=1.57 effort=10 velocity=1.0; origin xyz=0 -0.24462 0 rpy=0 0 0 -> xyz=0 0 -0.2407 rpy=0 0 0
- joint right_shoulder_pitch_joint: axis 1 0 0 -> 0 1 0; limit lower=-1.57 upper=1.57 effort=30 velocity=1.0 -> lower=-1.57 upper=1.57 effort=10 velocity=1.0; origin xyz=-0.0754 0.36378 0 rpy=0 0 0 -> xyz=0 -0.0793 -0.36378 rpy=0 0 0
- joint right_shoulder_roll_joint: axis 0 0 -1 -> 1 0 0; limit lower=-0.4 upper=3.14 effort=30 velocity=1.0 -> lower=-1.57 upper=1.57 effort=10 velocity=1.0; origin xyz=-0.17412 0 0 rpy=0 0 0 -> xyz=0 -0.1702 0 rpy=0 0 0
- joint right_shoulder_yaw_joint: axis 0 1 0 -> 0 0 1; limit lower=-1.57 upper=1.57 effort=30 velocity=1.0 -> lower=-1.57 upper=1.57 effort=10 velocity=1.0; origin xyz=0 -0.073 0 rpy=0 0 0 -> xyz=0 0 -0.0773 rpy=0 0 0
- joint right_wrist_pitch_joint: axis 1 0 0 -> 0 1 0; limit lower=-1.57 upper=1.57 effort=30 velocity=1.0 -> lower=-1.57 upper=1.57 effort=10 velocity=1.0; origin xyz=0 -0.15124 0 rpy=0 0 0 -> xyz=0.1472 0 0 rpy=0 0 0; parent right_wrist_yaw_link -> right_wrist_roll_link
- joint right_wrist_roll_joint: axis 0 0 1 -> 1 0 0; limit lower=-1.57 upper=1.57 effort=30 velocity=1.0 -> lower=-1.57 upper=1.57 effort=10 velocity=1.0; origin xyz=0 -0.07 0 rpy=0 0 0 -> xyz=0.0773 0 0 rpy=0 0 0; parent right_wrist_pitch_link -> right_elbow_pitch_link
- joint right_wrist_yaw_joint: axis 0 1 0 -> 0 0 1; limit lower=-1.57 upper=1.57 effort=30 velocity=1.0 -> lower=-1.57 upper=1.57 effort=10 velocity=1.0; origin xyz=0 -0.0732 0 rpy=0 0 0 -> xyz=0.0741 0 0 rpy=0 0 0; parent right_elbow_pitch_link -> right_wrist_pitch_link
