Commit message: major updates to model

File: dasl_robots/mk2/robots/mk2_arm.URDF (robot description, URDF)
Before this commit: robot mk2_arm, 8 links, 7 joints
Links:
- removed link right_elbow_pitch_link
- removed link right_shoulder_pitch_link
- removed link right_shoulder_roll_link
- removed link right_shoulder_yaw_link
- removed link right_wrist_pitch_link
- removed link right_wrist_roll_link
- removed link right_wrist_yaw_link
- removed link torso_roll_link
- added link base_link, mass 0.29334; collision mesh filename=package://mk2/meshes/base_link.STL; visual mesh filename=package://mk2/meshes/base_link.STL
- added link link_1, mass 0.14015; collision mesh filename=package://mk2/meshes/link_1.STL; visual mesh filename=package://mk2/meshes/link_1.STL
- added link link_2, mass 0.063501; collision mesh filename=package://mk2/meshes/link_2.STL; visual mesh filename=package://mk2/meshes/link_2.STL
- added link link_3, mass 0.234264171591375; collision mesh filename=package://mk2/meshes/link_3.STL; visual mesh filename=package://mk2/meshes/link_3.STL
- added link link_4, mass 0.0687829534109676; collision mesh filename=package://mk2/meshes/link_4.STL; visual mesh filename=package://mk2/meshes/link_4.STL
- added link link_5, mass 0.14324; collision mesh filename=package://mk2/meshes/link_5.STL; visual mesh filename=package://mk2/meshes/link_5.STL
- added link link_6, mass 0.043905; collision mesh filename=package://mk2/meshes/link_6.STL; visual mesh filename=package://mk2/meshes/link_6.STL
- added link link_7, mass 0.082562; collision mesh filename=package://mk2/meshes/link_7.STL; visual mesh filename=package://mk2/meshes/link_7.STL
Joints:
- removed joint right_elbow_pitch_joint
- removed joint right_shoulder_pitch_joint
- removed joint right_shoulder_roll_joint
- removed joint right_shoulder_yaw_joint
- removed joint right_wrist_pitch_joint
- removed joint right_wrist_roll_joint
- removed joint right_wrist_yaw_joint
- added joint joint_1: type revolute, parent base_link, child link_1, origin xyz=0 -0.0754 -0.57098 rpy=0 0 0, axis 0 1 0, limit lower=-1.57 upper=1.57 effort=10 velocity=2
- added joint joint_2: type revolute, parent link_1, child link_2, origin xyz=0 -0.17412 0 rpy=0 0 0, axis 1 0 0, limit lower=-1.57 upper=1.57 effort=10 velocity=2
- added joint joint_3: type revolute, parent link_2, child link_3, origin xyz=0 0 -0.07335 rpy=0 0 0, axis 0 0 1, limit lower=-1.57 upper=1.57 effort=10 velocity=2
- added joint joint_4: type revolute, parent link_3, child link_4, origin xyz=0 0 -0.24463 rpy=0 0 0, axis 0 1 0, limit lower=-1.57 upper=1.57 effort=10 velocity=2
- added joint joint_5: type revolute, parent link_4, child link_5, origin xyz=0.07335 0 0 rpy=0 0 0, axis 1 0 0, limit lower=-1.57 upper=1.57 effort=10 velocity=2
- added joint joint_6: type revolute, parent link_5, child link_6, origin xyz=0.1511 0 0 rpy=0 0 0, axis 0 1 0, limit lower=-1.57 upper=1.57 effort=10 velocity=2
- added joint joint_7: type revolute, parent link_6, child link_7, origin xyz=0.0741 0 0 rpy=0 0 0, axis 0 0 1, limit lower=-1.57 upper=1.57 effort=10 velocity=2

Commit message: updates to moveit config

File: dasl_robots/mk2/robots/mk2_arm.URDF (robot description, URDF)
Before this commit: robot mk2_arm, 8 links, 7 joints
Links:
- removed link base_link
- added link right_index_yaw_link, mass 0.018344; collision mesh filename=package://mk2/meshes/right_index_yaw_link.STL; visual mesh filename=package://mk2/meshes/right_index_yaw_link.STL
- added link right_palm_link, mass 0.284273788575286; collision mesh filename=package://mk2/meshes/right_palm_link.STL; visual mesh filename=package://mk2/meshes/right_palm_link.STL
- added link right_ring_yaw_link, mass 0.018344; collision mesh filename=package://mk2/meshes/right_ring_yaw_link.STL; visual mesh filename=package://mk2/meshes/right_ring_yaw_link.STL
- added link right_thumb_pitch_link, mass 0.0183440404710099; collision mesh filename=package://mk2/meshes/right_thumb_pitch_link.STL; visual mesh filename=package://mk2/meshes/right_thumb_pitch_link.STL
- added link right_thumb_roll_link, mass 0.0873520756053402; collision mesh filename=package://mk2/meshes/right_thumb_roll_link.STL; visual mesh filename=package://mk2/meshes/right_thumb_roll_link.STL
- added link torso_base_link, mass 0.13049; collision mesh filename=package://mk2/meshes/torso_base_link.STL; visual mesh filename=package://mk2/meshes/torso_base_link.STL
- added link torso_pitch_link, mass 0.214939247105387; collision mesh filename=package://mk2/meshes/torso_pitch_link.STL; visual mesh filename=package://mk2/meshes/torso_pitch_link.STL
- added link torso_roll_link, mass 0.293335697547887; collision mesh filename=package://mk2/meshes/torso_roll_link.STL; visual mesh filename=package://mk2/meshes/torso_roll_link.STL
- added link torso_yaw_link, mass 0.312439405406119; collision mesh filename=package://mk2/meshes/torso_yaw_link.STL; visual mesh filename=package://mk2/meshes/torso_yaw_link.STL
- link link_1: mass 0.14015 -> 0.140151957793056
- link link_2: mass 0.063501 -> 0.0635014085504459
- link link_3: mass 0.234264171591375 -> 0.23426
- link link_5: mass 0.14324 -> 0.143237868687531
- link link_6: mass 0.043905 -> 0.043905125184929
- link link_7: mass 0.082562 -> 0.0825624287077353
Joints:
- added joint right_index_yaw_joint: type revolute, parent right_palm_link, child right_index_yaw_link, origin xyz=0.16732 0 0.019252 rpy=0 0 0, axis 0 0 1, limit lower=-1.57 upper=1.57 effort=10 velocity=2
- added joint right_palm_joint: type fixed, parent link_7, child right_palm_link, origin xyz=0.051249 0 0 rpy=0 0 0, axis 1 0 0
- added joint right_ring_yaw_joint: type revolute, parent right_palm_link, child right_ring_yaw_link, origin xyz=0.16732 0 -0.0039672 rpy=0 0 0.042687, axis 0 0 1, limit lower=-1.57 upper=1.57 effort=10 velocity=2
- added joint right_thumb_pitch_joint: type revolute, parent right_thumb_roll_link, child right_thumb_pitch_link, origin xyz=0.023788 0 0.056923 rpy=0 0 0, axis 0 1 0, limit lower=-1.57 upper=1.57 effort=10 velocity=2
- added joint right_thumb_roll_joint: type revolute, parent right_palm_link, child right_thumb_roll_link, origin xyz=0.060596 0 0.015285 rpy=0 0 0, axis 1 0 0, limit lower=-1.57 upper=1.57 effort=10 velocity=2
- added joint torso_pitch_joint: type revolute, parent torso_yaw_link, child torso_pitch_link, origin xyz=0 0 -0.1065 rpy=0 0 0, axis 0 1 0, limit lower=-1.57 upper=1.57 effort=10 velocity=2
- added joint torso_roll_joint: type revolute, parent torso_pitch_link, child torso_roll_link, origin xyz=0 0 -0.08 rpy=0 0 0, axis 1 0 0, limit lower=-1.57 upper=1.57 effort=10 velocity=2
- added joint torso_yaw_joint: type revolute, parent torso_base_link, child torso_yaw_link, origin xyz=0 0 -0.0207 rpy=0 0 0, axis 0 0 1, limit lower=-1.57 upper=1.57 effort=10 velocity=2
- joint joint_1: origin xyz=0 -0.0754 -0.57098 rpy=0 0 0 -> xyz=0 -0.0754 -0.36378 rpy=0 0 0; parent base_link -> torso_roll_link
