Commit message: moveit changes

File: hdt/hdt_common/urdf/mk2.URDF (robot description, URDF)
Before this commit: robot mk2, 16 links, 15 joints
Links:
- removed link right_elbow_pitch_link
- removed link right_shoulder_pitch_link
- removed link right_shoulder_roll_link
- removed link right_shoulder_yaw_link
- removed link right_wrist_pitch_link
- removed link right_wrist_roll_link
- removed link right_wrist_yaw_link
- added link link_1, mass 0.140151957793056; collision mesh filename=package://mk2/meshes/link_1.STL; visual mesh filename=package://mk2/meshes/link_1.STL
- added link link_2, mass 0.0635014085504459; collision mesh filename=package://mk2/meshes/link_2.STL; visual mesh filename=package://mk2/meshes/link_2.STL
- added link link_3, mass 0.23426; collision mesh filename=package://mk2/meshes/link_3.STL; visual mesh filename=package://mk2/meshes/link_3.STL
- added link link_4, mass 0.0687829534109676; collision mesh filename=package://mk2/meshes/link_4.STL; visual mesh filename=package://mk2/meshes/link_4.STL
- added link link_5, mass 0.143237868687531; collision mesh filename=package://mk2/meshes/link_5.STL; visual mesh filename=package://mk2/meshes/link_5.STL
- added link link_6, mass 0.043905125184929; collision mesh filename=package://mk2/meshes/link_6.STL; visual mesh filename=package://mk2/meshes/link_6.STL
- added link link_7, mass 0.0825624287077353; collision mesh filename=package://mk2/meshes/link_7.STL; visual mesh filename=package://mk2/meshes/link_7.STL
- link right_index_yaw_link: mass 0.0183440339634614 -> 0.018344
- link right_palm_link: mass 0.28427392143233 -> 0.284273788575286
- link right_ring_yaw_link: mass 0.0183440282672802 -> 0.018344
- link right_thumb_pitch_link: mass 0.0183440323230481 -> 0.0183440404710099
- link right_thumb_roll_link: mass 0.0873520694654447 -> 0.0873520756053402
- link torso_base_link: mass 0.130487655760344 -> 0.13049
- link torso_pitch_link: mass 0.214939253072605 -> 0.214939247105387
- link torso_yaw_link: mass 0.312439405406118 -> 0.312439405406119
Joints:
- removed joint right_elbow_pitch_joint
- removed joint right_shoulder_pitch_joint
- removed joint right_shoulder_roll_joint
- removed joint right_shoulder_yaw_joint
- removed joint right_wrist_pitch_joint
- removed joint right_wrist_roll_joint
- removed joint right_wrist_yaw_joint
- added joint joint_1: type revolute, parent torso_roll_link, child link_1, origin xyz=0 -0.0754 -0.36378 rpy=0 0 0, axis 0 1 0, limit lower=-1.57 upper=1.57 effort=10 velocity=2
- added joint joint_2: type revolute, parent link_1, child link_2, origin xyz=0 -0.17412 0 rpy=0 0 0, axis 1 0 0, limit lower=-1.57 upper=1.57 effort=10 velocity=2
- added joint joint_3: type revolute, parent link_2, child link_3, origin xyz=0 0 -0.07335 rpy=0 0 0, axis 0 0 1, limit lower=-1.57 upper=1.57 effort=10 velocity=2
- added joint joint_4: type revolute, parent link_3, child link_4, origin xyz=0 0 -0.24463 rpy=0 0 0, axis 0 1 0, limit lower=-1.57 upper=1.57 effort=10 velocity=2
- added joint joint_5: type revolute, parent link_4, child link_5, origin xyz=0.07335 0 0 rpy=0 0 0, axis 1 0 0, limit lower=-1.57 upper=1.57 effort=10 velocity=2
- added joint joint_6: type revolute, parent link_5, child link_6, origin xyz=0.1511 0 0 rpy=0 0 0, axis 0 1 0, limit lower=-1.57 upper=1.57 effort=10 velocity=2
- added joint joint_7: type revolute, parent link_6, child link_7, origin xyz=0.0741 0 0 rpy=0 0 0, axis 0 0 1, limit lower=-1.57 upper=1.57 effort=10 velocity=2
- joint right_index_yaw_joint: limit lower=-1.57 upper=1.57 effort=10 velocity=1.0 -> lower=-1.57 upper=1.57 effort=10 velocity=2; origin xyz=0.0696 0 0.0193 rpy=0 0 0 -> xyz=0.16732 0 0.019252 rpy=0 0 0
- joint right_palm_joint: axis 0 0 0 -> 1 0 0; origin xyz=0.1489 0 0 rpy=0 0 0 -> xyz=0.051249 0 0 rpy=0 0 0; parent right_wrist_yaw_link -> link_7
- joint right_ring_yaw_joint: limit lower=-1.57 upper=1.57 effort=10 velocity=1.0 -> lower=-1.57 upper=1.57 effort=10 velocity=2; origin xyz=0.0696 0 -0.0039 rpy=0 0 0 -> xyz=0.16732 0 -0.0039672 rpy=0 0 0.042687
- joint right_thumb_pitch_joint: limit lower=-1.57 upper=1.57 effort=10 velocity=1.0 -> lower=-1.57 upper=1.57 effort=10 velocity=2; origin xyz=-0.013307 0 0.05692 rpy=0 0 0 -> xyz=0.023788 0 0.056923 rpy=0 0 0
- joint right_thumb_roll_joint: limit lower=-1.57 upper=1.57 effort=10 velocity=1.0 -> lower=-1.57 upper=1.57 effort=10 velocity=2; origin xyz=0 0 0.0153 rpy=0 0 0 -> xyz=0.060596 0 0.015285 rpy=0 0 0
- joint torso_pitch_joint: axis 0 -1 0 -> 0 1 0; limit lower=-1.57 upper=1.57 effort=10 velocity=1.0 -> lower=-1.57 upper=1.57 effort=10 velocity=2
- joint torso_roll_joint: limit lower=-1.57 upper=1.57 effort=10 velocity=1.0 -> lower=-1.57 upper=1.57 effort=10 velocity=2
- joint torso_yaw_joint: axis 0 0 -1 -> 0 0 1; limit lower=-1.57 upper=1.57 effort=10 velocity=1.0 -> lower=-1.57 upper=1.57 effort=10 velocity=2

Commit message: cleaned up mk2_controller

File: hdt/hdt_common/urdf/mk2.URDF (robot description, URDF)
Before this commit: robot mk2, 16 links, 15 joints
Links:
- link link_1: geometry collision mesh filename=package://hdt_common/meshes/link_1.STL; visual mesh filename=package://hdt_common/meshes/link_1.STL
- link link_2: geometry collision mesh filename=package://hdt_common/meshes/link_2.STL; visual mesh filename=package://hdt_common/meshes/link_2.STL
- link link_3: geometry collision mesh filename=package://hdt_common/meshes/link_3.STL; visual mesh filename=package://hdt_common/meshes/link_3.STL
- link link_4: geometry collision mesh filename=package://hdt_common/meshes/link_4.STL; visual mesh filename=package://hdt_common/meshes/link_4.STL
- link link_5: geometry collision mesh filename=package://hdt_common/meshes/link_5.STL; visual mesh filename=package://hdt_common/meshes/link_5.STL
- link link_6: geometry collision mesh filename=package://hdt_common/meshes/link_6.STL; visual mesh filename=package://hdt_common/meshes/link_6.STL
- link link_7: geometry collision mesh filename=package://hdt_common/meshes/link_7.STL; visual mesh filename=package://hdt_common/meshes/link_7.STL
- link right_index_yaw_link: geometry collision mesh filename=package://hdt_common/meshes/right_index_yaw_link.STL; visual mesh filename=package://hdt_common/meshes/right_index_yaw_link.STL
- link right_palm_link: geometry collision mesh filename=package://hdt_common/meshes/right_palm_link.STL; visual mesh filename=package://hdt_common/meshes/right_palm_link.STL
- link right_ring_yaw_link: geometry collision mesh filename=package://hdt_common/meshes/right_ring_yaw_link.STL; visual mesh filename=package://hdt_common/meshes/right_ring_yaw_link.STL
- link right_thumb_pitch_link: geometry collision mesh filename=package://hdt_common/meshes/right_thumb_pitch_link.STL; visual mesh filename=package://hdt_common/meshes/right_thumb_pitch_link.STL
- link right_thumb_roll_link: geometry collision mesh filename=package://hdt_common/meshes/right_thumb_roll_link.STL; visual mesh filename=package://hdt_common/meshes/right_thumb_roll_link.STL
- link torso_base_link: geometry collision mesh filename=package://hdt_common/meshes/torso_base_link.STL; visual mesh filename=package://hdt_common/meshes/torso_base_link.STL
- link torso_pitch_link: geometry collision mesh filename=package://hdt_common/meshes/torso_pitch_link.STL; visual mesh filename=package://hdt_common/meshes/torso_pitch_link.STL
- link torso_roll_link: geometry collision mesh filename=package://hdt_common/meshes/torso_roll_link.STL; visual mesh filename=package://hdt_common/meshes/torso_roll_link.STL
- link torso_yaw_link: geometry collision mesh filename=package://hdt_common/meshes/torso_yaw_link.STL; visual mesh filename=package://hdt_common/meshes/torso_yaw_link.STL

Commit message: added torso to ik

File: hdt/hdt_common/urdf/mk2.URDF (robot description, URDF)
Before this commit: robot mk2, 16 links, 15 joints
Joints:
- joint torso_pitch_joint: axis 0 1 0 -> 0 -1 0
- joint torso_yaw_joint: axis 0 0 1 -> 0 0 -1
